Commit message: simulate wheels

File: sapien_google_robot/googlerobot_description/meta_sim.urdf (robot description, URDF)
Before this commit: robot meta, 34 links, 33 joints
Links:
- added link link_rear_wheel_left; collision mesh filename=coarse_meshes/link_rear_wheel.glb; visual mesh filename=coarse_meshes/link_rear_wheel.glb
- added link link_rear_wheel_right; collision mesh filename=coarse_meshes/link_rear_wheel.glb; visual mesh filename=coarse_meshes/link_rear_wheel.glb
- link link_base: geometry collision mesh filename=coarse_meshes/link_base_0.glb; collision mesh filename=coarse_meshes/link_base_1.glb
Joints:
- added joint joint_rear_wheel_left: type continuous, parent link_base, child link_rear_wheel_left, origin xyz=-0.338371 0.094989 -0.029296 rpy=0 0 0, axis 0 1 0, limit lower=-inf upper=inf effort=10.0 velocity=12.9
- added joint joint_rear_wheel_right: type continuous, parent link_base, child link_rear_wheel_right, origin xyz=-0.338371 -0.094989 -0.029296 rpy=0 0 0, axis 0 1 0, limit lower=-inf upper=inf effort=10.0 velocity=12.9
