Commit message: process collision & visual

File: sapien_google_robot/googlerobot_description/meta_sim_fix_wheel.urdf (robot description, URDF)
Before this commit: robot meta, 36 links, 35 joints
Links:
- link link_base: geometry collision mesh filename=collision_meshes/link_base.glb; visual mesh filename=visual_meshes/link_base.glb
- link link_bicep: geometry collision mesh filename=collision_meshes/link_bicep.glb; visual mesh filename=visual_meshes/link_bicep.glb
- link link_elbow: geometry collision mesh filename=collision_meshes/link_elbow.glb; visual mesh filename=visual_meshes/link_elbow.glb
- link link_finger_left: geometry collision mesh filename=collision_meshes/link_finger_base.glb; visual mesh filename=visual_meshes/link_finger_base.glb
- link link_finger_nail_left: geometry visual mesh filename=visual_meshes/link_finger_nail.glb
- link link_finger_nail_right: geometry visual mesh filename=visual_meshes/link_finger_nail.glb
- link link_finger_right: geometry collision mesh filename=collision_meshes/link_finger_base.glb; visual mesh filename=visual_meshes/link_finger_base.glb
- link link_finger_tip_left: geometry collision mesh filename=collision_meshes/link_finger_tip.glb; visual mesh filename=visual_meshes/link_finger_tip.glb
- link link_finger_tip_right: geometry collision mesh filename=collision_meshes/link_finger_tip.glb; visual mesh filename=visual_meshes/link_finger_tip.glb
- link link_forearm: geometry collision mesh filename=collision_meshes/link_forearm.glb; visual mesh filename=visual_meshes/link_forearm.glb
- link link_gripper: geometry collision mesh filename=collision_meshes/link_gripper.glb; visual mesh filename=visual_meshes/link_gripper.glb
- link link_head_pan: geometry collision mesh filename=collision_meshes/link_head_pan.glb; visual mesh filename=visual_meshes/link_head_pan.glb
- link link_head_tilt: geometry collision mesh filename=collision_meshes/link_head_tilt.glb; visual mesh filename=visual_meshes/link_head_tilt.glb
- link link_rear_wheel_left: geometry collision mesh filename=collision_meshes/link_rear_wheel.glb; visual mesh filename=visual_meshes/link_rear_wheel.glb
- link link_rear_wheel_right: geometry collision mesh filename=collision_meshes/link_rear_wheel.glb; visual mesh filename=visual_meshes/link_rear_wheel.glb
- link link_shoulder: geometry collision mesh filename=collision_meshes/link_shoulder.glb; visual mesh filename=visual_meshes/link_shoulder.glb
- link link_torso: geometry collision mesh filename=collision_meshes/link_torso.glb; visual mesh filename=visual_meshes/link_torso.glb
- link link_wheel_left: geometry collision mesh filename=collision_meshes/link_wheel.glb; visual mesh filename=visual_meshes/link_wheel.glb
- link link_wheel_right: geometry collision mesh filename=collision_meshes/link_wheel.glb; visual mesh filename=visual_meshes/link_wheel.glb
- link link_wrist: geometry collision mesh filename=collision_meshes/link_wrist.glb; visual mesh filename=visual_meshes/link_wrist.glb
